File: Starbie/Starbie.kicad_sch (KiCad schematic)
At the start: 7 parts, among them J1 Conn_01x04_Pin, J2 Conn_01x08_Pin, SW1 SW_Push, SW2 SW_Push, U1 XIAO-ESP32-C3-SMD, U2 DHT11

Commit message: feat- added piezo buzzer to PCB
Parts:
- added BZ1: Buzzer, Buzzer_Beeper:Buzzer_12x9.5RM7.6, symbol Device:Buzzer
- added R2: 100, Resistor_THT:R_Axial_DIN0204_L3.6mm_D1.6mm_P7.62mm_Horizontal, symbol Device:R_US
Connections:
- net DIO 2: no longer U1.3 (D2)
- net DIO 3: no longer U1.4 (D3)
- net GND: now also R2.1
- net GPIO 20: now reaches U1.8 (D7)
- net GPIO 20: now also BZ1.1 (+)
- new net: BZ1.2 (-), R2.2
- new net GPIO 2: U1.3 (D2)
- new net GPIO 3: U1.4 (D3)
- no-connect marks 12 -> 11
