File: Starbie/_restore_backup_2026-10-10T14-58-09-723/Starbie.kicad_pcb (KiCad board)
At the start: 2 copper layers, 130.6 x 90.5 mm, 10 parts, among them J1 Conn_01x04_Pin, J2 Conn_01x08_Pin, SW1 SW_Push, SW2 SW_Push, U1 XIAO-ESP32-C3-SMD, U2 DHT11

Commit message: feat: add volume control to the PCB
Users now can adjust the volume of the Starbie  via a potentiometer connected to the buzzer.
Parts:
- removed RV2: R_Potentiometer_US, Potentiometer_THT:Potentiometer_ACP_CA9-V10_Vertical
- added R2: 100, Resistor_THT:R_Axial_DIN0204_L3.6mm_D1.6mm_P7.62mm_Horizontal, F.Cu at (171.0, 99.6)
Connections:
- BZ1 pad 1: Net-(BZ1-+) -> /GPIO 20
- BZ1 pad 2: GND -> Net-(BZ1--)
Routing:
- net /GPIO 20: track 56.1 -> 14.2 mm
- net Net-(BZ1--): track 0.00 -> 26.3 mm
- net Net-(BZ1-+): track 17.1 -> 0.00 mm
Other:
- board text removed: "Volume Control"
Changed lines of the file:
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@@
 		(tags "Resistor Axial_DIN0204 series Axial Horizontal pin pitch 7.62mm 0.167W length 3.6mm diameter 1.6mm")
 		(property "Reference" "R1"
-			(at 3.81 3 0)
+			(at 3.81 -1.92 0)
 			(layer "F.SilkS")
 			(effects
@@
 		)
 		(property "Value" "10k"
-			(at 8.81 1.92 0)
+			(at 3.81 1.92 0)
 			(layer "F.Fab")
 			(effects
@@
 			(layers "*.Cu" "*.Mask")
 			(remove_unused_layers no)
-			(net "Net-(BZ1-+)")
+			(net "/GPIO 20")
 			(pinfunction "+_1")
 			(pintype "passive")
@@
 			(layers "*.Cu" "*.Mask")
 			(remove_unused_layers no)
-			(net "GND")
+			(net "Net-(BZ1--)")
 			(pinfunction "-_2")
 			(pintype "passive")
 		)
 		(embedded_fonts no)
-		(model "${KICAD10_3DMODEL_DIR}/Buzzer_Beeper.3dshapes/Buzzer_12x9.5RM7.6.step"
+		(model "${KISYS3DMOD}/Buzzer_Beeper.3dshapes/Buzzer_12x9.5RM7.6.wrl"
 			(offset
 				(xyz 0 0 0)
@@
 		)
 	)
-	(footprint "Potentiometer_THT:Potentiometer_ACP_CA9-V10_Vertical"
+	(footprint "Resistor_THT:R_Axial_DIN0204_L3.6mm_D1.6mm_P7.62mm_Horizontal"
 		(layer "F.Cu")
-		(at 160 92.5)
-		(descr "Potentiometer, vertical, ACP CA9-V10, http://www.acptechnologies.com/wp-content/uploads/2017/05/02-ACP-CA9-CE9.pdf")
-		(tags "Potentiometer vertical ACP CA9-V10")
-		(property "Reference" "RV2"
-			(at 5 -8.65 0)
+		(at 170.975 99.625)
+		(descr "Resistor, Axial_DIN0204 series, Axial, Horizontal, pin pitch=7.62mm, 0.167W, length*diameter=3.6*1.6mm^2, http://cdn-reichelt.de/documents/datenblatt/B400/1_4W%23YAG.pdf")
+		(tags "Resistor Axial_DIN0204 series Axial Horizontal pin pitch 7.62mm 0.167W length 3.6mm diameter 1.6mm")
+		(property "Reference" "R2"
+			(at 3.81 -1.92 0)
 			(layer "F.SilkS")
 			(effects
@@
 			)
 		)
-		(property "Value" "R_Potentiometer_US"
-			(at 5 7.5 0)
+		(property "Value" "100"
+			(at 3.81 1.92 0)
 			(layer "F.Fab")
 			(effects
@@
 			)
 		)
-		(property "Description" "Potentiometer, US symbol"
+		(property "Description" "Resistor, US symbol"
 			(at 0 0 0)
 			(layer "F.Fab")
@@
 			)
 		)
-		(property "KiLib_Generator" "potentiometer/THT"
+		(property "KiLib_Generator" "resistor/THT"
 			(at 0 0 0)
 			(layer "F.SilkS")
@@
 			)
 		)
-		(property "Sim.Device" "R"
-			(at 0 0 0)
-			(unlocked yes)
-			(layer "F.Fab")
-			(hide yes)
-			(effects
-				(font
-					(size 1 1)
-					(thickness 0.15)
-				)
-			)
-		)
-		(property "Sim.Type" "POT"
-			(at 0 0 0)
-			(unlocked yes)
-			(layer "F.Fab")
-			(hide yes)
-			(effects
-				(font
-					(size 1 1)
-					(thickness 0.15)
-				)
-			)
-		)
-		(property "Sim.Pins" "1=r0 2=wiper 3=r1"
-			(at 0 0 0)
-			(unlocked yes)
-			(layer "F.Fab")
-			(hide yes)
-			(effects
-				(font
-					(size 1 1)
-					(thickness 0.15)
-				)
-			)
-		)
-		(property ki_fp_filters "Potentiometer*")
+		(property ki_fp_filters "R_*")
 		(sheetname "/")
 		(sheetfile "Starbie.kicad_sch")
@@
 			(unit
 				(name "A")
-				(pins "1" "3" "2")
+				(pins "1" "2")
 			)
 		)
@@
 		(duplicate_pad_numbers_are_jumpers no)
 		(fp_line
-			(start -0.11 -7.51)
-			(end 10.11 -7.51)
-			(stroke
-				(width 0.12)
-				(type solid)
-			)
-			(layer "F.SilkS")
-		)
-		(fp_line
-			(start -0.11 -6.396)
-			(end -0.11 -7.51)
+			(start 0.94 0)
+			(end 1.89 0)
 			(stroke
 				(width 0.12)
@@
 		)
 		(fp_line
-			(start -0.11 -1.396)
-			(end -0.11 -3.604)
+			(start 6.68 0)
+			(end 5.73 0)
 			(stroke
 				(width 0.12)
@@
 			(layer "F.SilkS")
 		)
-		(fp_line
-			(start -0.11 2.51)
-			(end -0.11 1.396)
+		(fp_rect
+			(start 1.89 -0.92)
+			(end 5.73 0.92)
 			(stroke
 				(width 0.12)
 				(type solid)
 			)
+			(fill no)
 			(layer "F.SilkS")
 		)
-		(fp_line
-			(start 10.11 -7.51)
-			(end 10.11 -3.896)
+		(fp_rect
+			(start -0.95 -1.05)
+			(end 8.57 1.05)
 			(stroke
-				(width 0.12)
+				(width 0.05)
 				(type solid)
 			)
-			(layer "F.SilkS")
+			(fill no)
+			(layer "F.CrtYd")
 		)
 		(fp_line
-			(start 10.11 -1.104)
-			(end 10.11 2.51)
+			(start 0 0)
+			(end 2.01 0)
 			(stroke
-				(width 0.12)
+				(width 0.1)
 				(type solid)
 			)
-			(layer "F.SilkS")
+			(layer "F.Fab")
 		)
 		(fp_line
-			(start 10.11 2.51)
-			(end -0.11 2.51)
-			(stroke
-				(width 0.12)
-				(type solid)
-			)
-			(layer "F.SilkS")
-		)
-		(fp_rect
-			(start -1.42 -7.65)
-			(end 11.42 2.66)
-			(stroke
-				(width 0.05)
-				(type solid)
-			)
-			(fill no)
-			(layer "F.CrtYd")
-		)
-		(fp_rect
-			(start 0 -7.4)
-			(end 10 2.4)
+			(start 7.62 0)
+			(end 5.61 0)
 			(stroke
 				(width 0.1)
 				(type solid)
 			)
-			(fill no)
 			(layer "F.Fab")
 		)
-		(fp_circle
-			(center 5 -2.5)
-			(end 6.05 -2.5)
+		(fp_rect
+			(start 2.01 -0.8)
+			(end 5.61 0.8)
 			(stroke
 				(width 0.1)
@@
 		)
 		(fp_text user "${REFERENCE}"
-			(at 1 -2.5 90)
+			(at 3.81 0 0)
 			(layer "F.Fab")
 			(effects
 				(font
-					(size 1 1)
-					(thickness 0.15)
+					(size 0.72 0.72)
+					(thickness 0.108)
 				)
 			)
@@
 		(pad "1" thru_hole circle
 			(at 0 0)
-			(size 2.34 2.34)
-			(drill 1.3)
+			(size 1.4 1.4)
+			(drill 0.7)
 			(layers "*.Cu" "*.Mask")
 			(remove_unused_layers no)
-			(net "/GPIO 20")
-			(pinfunction "1_1")
+			(net "GND")
 			(pintype "passive")
 		)
 		(pad "2" thru_hole circle
-			(at 10 -2.5)
-			(size 2.34 2.34)
-			(drill 1.3)
-			(layers "*.Cu" "*.Mask")
-			(remove_unused_layers no)
-			(net "Net-(BZ1-+)")
-			(pinfunction "2_2")
-			(pintype "passive")
-		)
-		(pad "3" thru_hole circle
-			(at 0 -5)
-			(size 2.34 2.34)
-			(drill 1.3)
+			(at 7.62 0)
+			(size 1.4 1.4)
+			(drill 0.7)
 			(layers "*.Cu" "*.Mask")
 			(remove_unused_layers no)
-			(net "GND")
-			(pinfunction "3_3")
+			(net "Net-(BZ1--)")
 			(pintype "passive")
 		)
 		(embedded_fonts no)
-		(model "${KICAD10_3DMODEL_DIR}/Potentiometer_THT.3dshapes/Potentiometer_ACP_CA9-V10_Vertical.step"
+		(model "${KICAD10_3DMODEL_DIR}/Resistor_THT.3dshapes/R_Axial_DIN0204_L3.6mm_D1.6mm_P7.62mm_Horizontal.step"
 			(offset
 				(xyz 0 0 0)
@@
 			(at 1 0 0)
 			(unlocked yes)
-			(layer "F.SilkS")
+			(layer "F.Fab")
 			(effects
 				(font
@@
 		(layer "Edge.Cuts")
 	)
-	(gr_text "Volume Control"
-		(at 160 100 0)
-		(layer "F.SilkS")
-		(effects
-			(font
-				(size 1 1)
-				(thickness 0.1)
-			)
-			(justify left bottom)
-		)
-	)
 	(segment
 		(start 127.04 59.77)
@@
 	)
 	(segment
-		(start 125 80)
-		(end 100 80)
+		(start 178.595 99.625)
+		(end 182.6 95.62)
 		(width 0.2)
 		(layer "F.Cu")
-		(net "/GPIO 2")
+		(net "Net-(BZ1--)")
 	)
 	(segment
-		(start 147.38 58.46)
-		(end 145.30237 58.46)
+		(start 182.6 95.62)
+		(end 182.6 75)
 		(width 0.2)
 		(layer "F.Cu")
-		(net "/GPIO 2")
+		(net "Net-(BZ1--)")
 	)
 	(segment
-		(start 145.30237 58.46)
-		(end 125 78.76237)
+		(start 168.62 68.62)
+		(end 175 75)
 		(width 0.2)
 		(layer "F.Cu")
-		(net "/GPIO 2")
-	)
-	(segment
-		(start 100 80)
-		(end 100 95)
-		(width 0.2)
-		(layer "F.Cu")
-		(net "/GPIO 2")
-	)
-	(segment
-		(start 112.46 107.46)
-		(end 112.46 114.92)
-		(width 0.2)
-		(layer "F.Cu")
-		(net "/GPIO 2")
-	)
-	(segment
-		(start 125 78.76237)
-		(end 125 80)
-		(width 0.2)
-		(layer "F.Cu")
-		(net "/GPIO 2")
+		(net "/GPIO 20")
 	)
 	(segment
-		(start 100 95)
-		(end 112.46 107.46)
+		(start 163.455 68.62)
+		(end 168.62 68.62)
 		(width 0.2)
 		(layer "F.Cu")
-		(net "/GPIO 2")
+		(net "/GPIO 20")
 	)
 	(segment
@@
 	)
 	(segment
-		(start 175 75)
-		(end 175 85)
-		(width 0.2)
-		(layer "B.Cu")
-		(net "Net-(BZ1-+)")
-	)
-	(segment
-		(start 175 85)
-		(end 170 90)
+		(start 125 80)
+		(end 100 80)
 		(width 0.2)
-		(layer "B.Cu")
-		(net "Net-(BZ1-+)")
+		(layer "F.Cu")
+		(net "/GPIO 2")
 	)
 	(segment
-		(start 162.62 68.62)
-		(end 162.62 72.62)
+		(start 147.38 58.46)
+		(end 145.30237 58.46)
 		(width 0.2)
 		(layer "F.Cu")
-		(net "/GPIO 20")
+		(net "/GPIO 2")
 	)
 	(segment
-		(start 160 95)
-		(end 160 92.5)
+		(start 145.30237 58.46)
+		(end 125 78.76237)
 		(width 0.2)
 		(layer "F.Cu")
-		(net "/GPIO 20")
+		(net "/GPIO 2")
 	)
 	(segment
-		(start 165 100)
-		(end 160 95)
+		(start 100 80)
+		(end 100 95)
 		(width 0.2)
 		(layer "F.Cu")
-		(net "/GPIO 20")
+		(net "/GPIO 2")
 	)
 	(segment
-		(start 175 85)
-		(end 175 100)
+		(start 112.46 107.46)
+		(end 112.46 114.92)
 		(width 0.2)
 		(layer "F.Cu")
-		(net "/GPIO 20")
+		(net "/GPIO 2")
 	)
 	(segment
-		(start 175 100)
-		(end 165 100)
+		(start 125 78.76237)
+		(end 125 80)
 		(width 0.2)
 		(layer "F.Cu")
-		(net "/GPIO 20")
+		(net "/GPIO 2")
 	)
 	(segment
-		(start 162.62 72.62)
-		(end 175 85)
+		(start 100 95)
+		(end 112.46 107.46)
 		(width 0.2)
 		(layer "F.Cu")
-		(net "/GPIO 20")
+		(net "/GPIO 2")
 	)
 	(zone
