File: Starbie/_restore_backup_2026-10-10T14-58-09-723/Starbie.kicad_sch (KiCad schematic)
At the start: 9 parts, among them J1 Conn_01x04_Pin, J2 Conn_01x08_Pin, SW1 SW_Push, SW2 SW_Push, U1 XIAO-ESP32-C3-SMD, U2 DHT11

Commit message: feat: add volume control to the PCB
Users now can adjust the volume of the Starbie  via a potentiometer connected to the buzzer.
Parts:
- RV2: footprint Potentiometer_THT:Potentiometer_ACP_CA9-V10_Vertical -> Potentiometer_THT:Potentiometer_Alps_RK09K_Single_Vertical
Changed lines of the file:
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@@
 			)
 		)
-		(property "Footprint" "Potentiometer_THT:Potentiometer_ACP_CA9-V10_Vertical"
+		(property "Footprint" "Potentiometer_THT:Potentiometer_Alps_RK09K_Single_Vertical"
 			(at 236.22 43.18 0)
 			(hide yes)
